Commit message: We can run full ur5e with gripper

File: robotiq_description/urdf/ur_to_robotiq_adapter.urdf.xacro (robot description, xacro)
@@ -12,5 +12,5 @@
           <origin xyz="0 0 0" rpy="0 0 0" />
           <geometry>
-            <mesh filename="package://robotiq_description/meshes/visual/ur_to_robotiq_adapter.dae"/>
+            <mesh filename="file://$(find robotiq_description)/meshes/visual/ur_to_robotiq_adapter.dae"/>
           </geometry>
         </visual>
@@ -18,5 +18,5 @@
           <origin xyz="0 0 0" rpy="0 0 0"/>
           <geometry>
-            <mesh filename="package://robotiq_description/meshes/collision/ur_to_robotiq_adapter.stl"/>
+            <mesh filename="file://$(find robotiq_description)/meshes/collision/ur_to_robotiq_adapter.stl"/>
           </geometry>
         </collision>
