Commit message: We can move gripper easy, but pointcloud doesn't work on gripper yet

File: robotiq_description/urdf/robotiq_2f_85_macro.urdf.xacro (robot description, xacro)
@@ -36,5 +36,5 @@
             </inertial>
         </link>
-        <!-- <joint name="${prefix}robotiq_85_left_knuckle_joint" type="revolute">
+        <joint name="${prefix}robotiq_85_left_knuckle_joint" type="revolute">
             <parent link="${prefix}robotiq_85_base_link" />
             <child link="${prefix}robotiq_85_left_knuckle_link" />
@@ -62,6 +62,6 @@
                     iyz="0" />
             </inertial>
-        </link> -->
-        <!-- <link name="${prefix}robotiq_85_right_knuckle_link">
+        </link>
+        <link name="${prefix}robotiq_85_right_knuckle_link">
             <visual>
                 <geometry>
@@ -291,5 +291,5 @@
             <origin xyz="-0.00563134 0.0 0.04718515" rpy="0 0 0" />
             <mimic joint="${prefix}robotiq_85_left_knuckle_joint" />
-        </joint> -->
+        </joint>
         <gazebo>
             <plugin name="gripper_control" filename="libcontrol_plugin.so" />
