Commit message: We fixed control scheme, pointclouds on the gripper, moved the camera so it matches with Isaac Sim, and got the lighting working for UR5

File: robotiq_description/urdf/robotiq_2f_85_gripper.urdf.xacro (robot description, xacro)
@@ -9,16 +9,3 @@
         <origin xyz="0 0 0" rpy="0 0 0" />
     </xacro:robotiq_gripper>
-    <!-- <gazebo>
-        <plugin name="no_physics" filename="libno_physics_plugin.so" />
-    </gazebo> -->
-    <gazebo>
-        <plugin filename="libgazebo_ros2_control.so" name="gazebo_ros2_control">
-            <parameters>
-                /home/kushtimusprime/cross_embodiment_test_ws/src/robotiq_driver/config/basic_controller.yaml
-            </parameters>
-        </plugin>
-    </gazebo>
-    <gazebo>
-        <plugin name="control" filename="libcontrol_plugin.so" />
-    </gazebo>
 </robot>

File: robotiq_description/urdf/robotiq_2f_85_macro.urdf.xacro (robot description, xacro)
@@ -1,13 +1,216 @@
 <?xml version="1.0"?>
 <robot xmlns:xacro="http://wiki.ros.org/xacro" name="robotiq_gripper">
-    <xacro:macro name="robotiq_gripper" params="prefix parent *origin">
-        <!-- ros2 control include
+    <xacro:macro name="robotiq_gripper" params="
+        name
+        prefix
+        parent
+        *origin
+        sim_ignition:=false
+        sim_isaac:=false
+        use_fake_hardware:=false
+        fake_sensor_commands:=false
+        include_ros2_control:=true
+        com_port:=/dev/ttyUSB0">
+        <!-- ros2 control include -->
         <xacro:include filename="$(find robotiq_description)/urdf/robotiq_gripper.ros2_control.xacro" />
+        <!-- if we are simulating or directly communicating with the gripper we need a ros2 control instance -->
         <xacro:if value="${include_ros2_control}">
-            <xacro:robotiq_gripper_ros2_control name="${name}" prefix="${prefix}"
-        sim_ignition="${sim_ignition}" sim_isaac="${sim_isaac}"
-        use_fake_hardware="${use_fake_hardware}" fake_sensor_commands="${fake_sensor_commands}"
-        com_port="${com_port}"/>
-        </xacro:if> -->
+            <xacro:robotiq_gripper_ros2_control
+                name="${name}" prefix="${prefix}"
+                sim_ignition="${sim_ignition}"
+                sim_isaac="${sim_isaac}"
+                use_fake_hardware="${use_fake_hardware}"
+                fake_sensor_commands="${fake_sensor_commands}"
+                com_port="${com_port}"/>
+        </xacro:if>
+        <link name="${prefix}robotiq_85_base_link">
+            <visual>
+                <geometry>
+                    <mesh filename="file://$(find robotiq_description)/meshes/visual/robotiq_base.dae" />
+                </geometry>
+            </visual>
+            <collision>
+                <geometry>
+                    <mesh filename="file://$(find robotiq_description)/meshes/collision/robotiq_base.stl" />
+                </geometry>
+            </collision>
+            <inertial>
+                <origin xyz="0.0 2.274e-05 0.03232288" rpy="0 0 0" />
+                <mass value="6.6320197e-01" />
+                <inertia ixx="5.1617816e-04" iyy="5.8802208e-04" izz="3.9462776e-04" ixy="2.936e-8" ixz="0.0" iyz="-3.2296e-7" />
+            </inertial>
+        </link>
+        <link name="${prefix}robotiq_85_left_knuckle_link">
+            <visual>
+                <geometry>
+                    <mesh filename="file://$(find robotiq_description)/meshes/visual/left_knuckle.dae" />
+                </geometry>
+            </visual>
+            <collision>
+                <geometry>
+                    <mesh filename="file://$(find robotiq_description)/meshes/collision/left_knuckle.stl" />
+                </geometry>
+            </collision>
+            <inertial>
+                <origin xyz="0.01213197 0.0002 -0.00058647" rpy="0 0 0" />
+                <mass value="1.384773208e-02" />
+                <inertia ixx="3.5232e-7" iyy="2.31944e-6" izz="2.23136e-6" ixy="0.0" ixz="1.1744e-7" iyz="0" />
+            </inertial>
+        </link>
+        <link name="${prefix}robotiq_85_right_knuckle_link">
+            <visual>
+                <geometry>
+                    <mesh filename="file://$(find robotiq_description)/meshes/visual/right_knuckle.dae" />
+                </geometry>
+            </visual>
+            <collision>
+                <geometry>
+                    <mesh filename="file://$(find robotiq_description)/meshes/collision/right_knuckle.stl" />
+                </geometry>
+            </collision>
+            <inertial>
+                <origin xyz="-0.01213197 0.0002 -0.00058647" rpy="0 0 0" />
+                <mass value="1.384773208e-02" />
+                <inertia ixx="3.5232e-7" iyy="2.31944e-6" izz="2.23136e-6" ixy="0.0" ixz="-1.1744e-7" iyz="0.0" />
+            </inertial>
+        </link>
+        <link name="${prefix}robotiq_85_left_finger_link">
+            <visual>
+                <geometry>
+                    <mesh filename="file://$(find robotiq_description)/meshes/visual/left_finger.dae" />
+                </geometry>
+            </visual>
+            <collision>
+                <geometry>
+                    <mesh filename="file://$(find robotiq_description)/meshes/collision/left_finger.stl" />
+                </geometry>
+            </collision>
+            <inertial>
+                <origin xyz="0.00346899 -0.00079447 0.01867121" rpy="0 0 0" />
+                <mass value="4.260376752e-02" />
+                <inertia ixx="1.385792000000000e-05" iyy="1.183208e-05" izz="5.19672e-06" ixy="0.0" ixz="-2.17264e-06" iyz="0.0" />
+            </inertial>
+        </link>
+        <link name="${prefix}robotiq_85_right_finger_link">
+            <visual>
+                <geometry>
+                    <mesh filename="file://$(find robotiq_description)/meshes/visual/right_finger.dae" />
+                </geometry>
+            </visual>
+            <collision>
+                <geometry>
+                    <mesh filename="file://$(find robotiq_description)/meshes/collision/right_finger.stl" />
+                </geometry>
+            </collision>
+            <inertial>
+                <origin xyz="-0.00346899 -5.53e-06 0.01867121" rpy="0 0 0" />
+                <mass value="4.260376752000000e-02" />
+                <inertia ixx="1.385792e-05" iyy="1.183208e-05" izz="5.19672e-06" ixy="0.0" ixz="2.17264e-06" iyz="0.0" />
+            </inertial>
+        </link>
+        <link name="${prefix}robotiq_85_left_inner_knuckle_link">
+            <visual>
+                <geometry>
+                    <mesh filename="file://$(find robotiq_description)/meshes/visual/left_inner_knuckle.dae" />
+                </geometry>
+            </visual>
+            <collision>
+                <geometry>
+                    <mesh filename="file://$(find robotiq_description)/meshes/collision/left_inner_knuckle.stl" />
+                </geometry>
+            </collision>
+            <inertial>
+                <origin xyz="0.01897699 0.00015001 0.02247101" rpy="0 0 0" />
+                <mass value="2.969376448e-02" />
+                <inertia ixx="9.57136e-06" iyy="8.69056e-06" izz="8.19144e-06" ixy="0.0" ixz="-3.93424e-06" iyz="0.0" />
+            </inertial>
+        </link>
+        <link name="${prefix}robotiq_85_right_inner_knuckle_link">
+            <visual>
+                <geometry>
+                    <mesh filename="file://$(find robotiq_description)/meshes/visual/right_inner_knuckle.dae" />
+                </geometry>
+            </visual>
+            <collision>
+                <geometry>
+                    <mesh filename="file://$(find robotiq_description)/meshes/collision/right_inner_knuckle.stl" />
+                </geometry>
+            </collision>
+            <inertial>
+                <origin xyz="-0.01926824 5.001e-05 0.02222178" rpy="0 0 0" />
+                <mass value="2.969376448e-02" />
+                <inertia ixx="9.42456e-06" iyy="8.69056e-06" izz="8.33824e-06" ixy="0.0" ixz="3.9636e-06" iyz="0.0" />
+            </inertial>
+        </link>
+        <link name="${prefix}robotiq_85_left_finger_tip_link">
+            <visual>
+                <geometry>
+                    <mesh filename="file://$(find robotiq_description)/meshes/visual/left_finger_tip.dae" />
+                </geometry>
+            </visual>
+            <collision>
+                <geometry>
+                    <mesh filename="file://$(find robotiq_description)/meshes/collision/left_finger_tip.stl" />
+                </geometry>
+                <surface>
+                    <friction>
+                    <ode>
+                        <mu1>100000.0</mu1>
+                        <mu2>100000.0</mu2>
+                    </ode>
+                    </friction>
+                    <contact>
+                    <ode>
+                        <kp>1e+5</kp>
+                        <kd>1</kd>
+                        <soft_cfm>0</soft_cfm>
+                        <soft_erp>0.2</soft_erp>
+                        <minDepth>0.002</minDepth>
+                        <maxVel>0</maxVel>
+                    </ode>
+                    </contact>
+                </surface>
+            </collision>
+            <inertial>
+                <origin xyz="-0.01456706 -0.0008 0.01649701" rpy="0 0 0" />
+                <mass value="4.268588744e-02" />
+                <inertia ixx="1.048152e-05" iyy="1.197888e-05" izz="4.22784e-06" ixy="0.0" ixz="3.5232e-6" iyz="0.0" />
+            </inertial>
+        </link>
+        <link name="${prefix}robotiq_85_right_finger_tip_link">
+            <visual>
+                <geometry>
+                    <mesh filename="file://$(find robotiq_description)/meshes/visual/right_finger_tip.dae" />
+                </geometry>
+            </visual>
+            <collision>
+                <geometry>
+                    <mesh filename="file://$(find robotiq_description)/meshes/collision/right_finger_tip.stl" />
+                </geometry>
+                <surface>
+                    <friction>
+                    <ode>
+                        <mu1>100000.0</mu1>
+                        <mu2>100000.0</mu2>
+                    </ode>
+                    </friction>
+                    <contact>
+                    <ode>
+                        <kp>1e+5</kp>
+                        <kd>1</kd>
+                        <soft_cfm>0</soft_cfm>
+                        <soft_erp>0.2</soft_erp>
+                        <minDepth>0.002</minDepth>
+                        <maxVel>0</maxVel>
+                    </ode>
+                    </contact>
+                </surface>
+            </collision>
+            <inertial>
+                <origin xyz="0.01456706 5e-05 0.01649701" rpy="0 0 0" />
+                <mass value="4.268588744e-02" />
+                <inertia ixx="1.048152e-05" iyy="1.197888e-05" izz="4.22784e-06" ixy="0.0" ixz="-3.5232e-06" iyz="0.0" />
+            </inertial>
+        </link>
         <joint name="${prefix}robotiq_85_base_joint" type="fixed">
             <parent link="${parent}" />
@@ -15,246 +218,10 @@
             <xacro:insert_block name="origin" />
         </joint>
-        <link name="${prefix}robotiq_85_base_link">
-            <visual>
-                <origin rpy="0 0 0" xyz="0 0 0"/>
-                <geometry>
-                    <mesh
-                        filename="file://$(find robotiq_description)/meshes/visual/robotiq_base.dae" />
-                </geometry>
-            </visual>
-            <collision>
-                <geometry>
-                    <mesh
-                        filename="file://$(find robotiq_description)/meshes/collision/robotiq_base.stl" />
-                </geometry>
-            </collision>
-            <inertial>
-                <origin xyz="0.0 2.274e-05 0.03232288" rpy="0 0 0" />
-                <mass value="6.6320197e-01" />
-                <inertia ixx="5.1617816e-04" iyy="5.8802208e-04" izz="3.9462776e-04" ixy="2.936e-8"
-                    ixz="0.0" iyz="-3.2296e-7" />
-            </inertial>
-        </link>
         <joint name="${prefix}robotiq_85_left_knuckle_joint" type="revolute">
             <parent link="${prefix}robotiq_85_base_link" />
             <child link="${prefix}robotiq_85_left_knuckle_link" />
+            <axis xyz="0 -1 0" />
             <origin xyz="0.03060114 0.0 0.05490452" rpy="0 0 0" />
-            <axis xyz="0 -1 0" />
             <limit lower="0.0" upper="0.8" velocity="0.5" effort="50" />
-            <safety_controller k_position="20" k_velocity="0.0"
-                soft_lower_limit="-6.133185307179586"
-                soft_upper_limit="6.133185307179586" />
-            <dynamics damping="0" friction="0" />
-        </joint>
-        <link name="${prefix}robotiq_85_left_knuckle_link">
-            <visual>
-                <origin rpy="0 0 0" xyz="0 0 0"/>
-                <geometry>
-                    <mesh
-                        filename="file://$(find robotiq_description)/meshes/visual/left_knuckle.dae" />
-                </geometry>
-            </visual>
-            <collision>
-                <geometry>
-                    <mesh
-                        filename="file://$(find robotiq_description)/meshes/collision/left_knuckle.stl" />
-                </geometry>
-            </collision>
-            <inertial>
-                <origin xyz="0.01213197 0.0002 -0.00058647" rpy="0 0 0" />
-                <mass value="1.384773208e-02" />
-                <inertia ixx="3.5232e-7" iyy="2.31944e-6" izz="2.23136e-6" ixy="0.0" ixz="1.1744e-7"
-                    iyz="0" />
-            </inertial>
-        </link>
-        <link name="${prefix}robotiq_85_right_knuckle_link">
-            <visual>
-                <origin rpy="0 0 0" xyz="0 0 0"/>
-                <geometry>
-                    <mesh
-                        filename="file://$(find robotiq_description)/meshes/visual/right_knuckle.dae" />
-                </geometry>
-            </visual>
-            <collision>
-                <geometry>
-                    <mesh
-                        filename="file://$(find robotiq_description)/meshes/collision/right_knuckle.stl" />
-                </geometry>
-            </collision>
-            <inertial>
-                <origin xyz="-0.01213197 0.0002 -0.00058647" rpy="0 0 0" />
-                <mass value="1.384773208e-02" />
-                <inertia ixx="3.5232e-7" iyy="2.31944e-6" izz="2.23136e-6" ixy="0.0"
-                    ixz="-1.1744e-7" iyz="0.0" />
-            </inertial>
-        </link>
-        <link name="${prefix}robotiq_85_left_finger_link">
-            <visual>
-                <origin rpy="0 0 0" xyz="0 0 0"/>
-                <geometry>
-                    <mesh
-                        filename="file://$(find robotiq_description)/meshes/visual/left_finger.dae" />
-                </geometry>
-            </visual>
-            <collision>
-                <geometry>
-                    <mesh
-                        filename="file://$(find robotiq_description)/meshes/collision/left_finger.stl" />
-                </geometry>
-            </collision>
-            <inertial>
-                <origin xyz="0.00346899 -0.00079447 0.01867121" rpy="0 0 0" />
-                <mass value="4.260376752e-02" />
-                <inertia ixx="1.385792000000000e-05" iyy="1.183208e-05" izz="5.19672e-06" ixy="0.0"
-                    ixz="-2.17264e-06" iyz="0.0" />
-            </inertial>
-        </link>
-        <link name="${prefix}robotiq_85_right_finger_link">
-            <visual>
-                <origin rpy="0 0 0" xyz="0 0 0"/>
-                <geometry>
-                    <mesh
-                        filename="file://$(find robotiq_description)/meshes/visual/right_finger.dae" />
-                </geometry>
-            </visual>
-            <collision>
-                <geometry>
-                    <mesh
-                        filename="file://$(find robotiq_description)/meshes/collision/right_finger.stl" />
-                </geometry>
-            </collision>
-            <inertial>
-                <origin xyz="-0.00346899 -5.53e-06 0.01867121" rpy="0 0 0" />
-                <mass value="4.260376752000000e-02" />
-                <inertia ixx="1.385792e-05" iyy="1.183208e-05" izz="5.19672e-06" ixy="0.0"
-                    ixz="2.17264e-06" iyz="0.0" />
-            </inertial>
-        </link>
-        <link name="${prefix}robotiq_85_left_inner_knuckle_link">
-            <visual>
-                <origin rpy="0 0 0" xyz="0 0 0"/>
-                <geometry>
-                    <mesh
-                        filename="file://$(find robotiq_description)/meshes/visual/left_inner_knuckle.dae" />
-                </geometry>
-            </visual>
-            <collision>
-                <geometry>
-                    <mesh
-                        filename="file://$(find robotiq_description)/meshes/collision/left_inner_knuckle.stl" />
-                </geometry>
-            </collision>
-            <inertial>
-                <origin xyz="0.01897699 0.00015001 0.02247101" rpy="0 0 0" />
-                <mass value="2.969376448e-02" />
-                <inertia ixx="9.57136e-06" iyy="8.69056e-06" izz="8.19144e-06" ixy="0.0"
-                    ixz="-3.93424e-06" iyz="0.0" />
-            </inertial>
-        </link>
-        <link name="${prefix}robotiq_85_right_inner_knuckle_link">
-            <visual>
-                <origin rpy="0 0 0" xyz="0 0 0"/>
-                <geometry>
-                    <mesh
-                        filename="file://$(find robotiq_description)/meshes/visual/right_inner_knuckle.dae" />
-                </geometry>
-            </visual>
-            <collision>
-                <geometry>
-                    <mesh
-                        filename="file://$(find robotiq_description)/meshes/collision/right_inner_knuckle.stl" />
-                </geometry>
-            </collision>
-            <inertial>
-                <origin xyz="-0.01926824 5.001e-05 0.02222178" rpy="0 0 0" />
-                <mass value="2.969376448e-02" />
-                <inertia ixx="9.42456e-06" iyy="8.69056e-06" izz="8.33824e-06" ixy="0.0"
-                    ixz="3.9636e-06" iyz="0.0" />
-            </inertial>
-        </link>
-        <link name="${prefix}robotiq_85_left_finger_tip_link">
-            <visual>
-                <origin rpy="0 0 0" xyz="0 0 0"/>
-                <geometry>
-                    <mesh
-                        filename="file://$(find robotiq_description)/meshes/visual/left_finger_tip.dae" />
-                </geometry>
-            </visual>
-            <collision>
-                <geometry>
-                    <mesh
-                        filename="file://$(find robotiq_description)/meshes/collision/left_finger_tip.stl" />
-                </geometry>
-                <surface>
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