Commit message: Made dummy end effector and now we can see the robot in RVIZ

File: gazebo_env/description/urdf/ur5e.urdf.xacro (robot description, xacro)
@@ -10,7 +10,8 @@
 https://github.com/ros-simulation/gazebo_ros_demos/blob/kinetic-devel/rrbot_description/urdf/rrbot.xacro
 -->
-<robot name="ur5e_robot"
+<robot name="2dof_robot"
     xmlns:xacro="http://ros.org/wiki/xacro">
-    <xacro:macro name="ur5e" params="parent *origin">
+    <xacro:macro name="ur5e">
+        <!-- <xacro:include filename="$(find gazebo_env)/urdf/d435.urdf.xacro" /> -->
         <material name="black">
             <color rgba="0.0 0.0 0.0 1.0" />
@@ -41,4 +42,13 @@
         </material>
         <!-- Used for fixing robot -->
+        <link name="world" />
+        <!-- <xacro:sensor_d435 parent="world">
+            <origin xyz="1.5 1.5 1" rpy="0 0.5235987756 -2.35619449" />
+        </xacro:sensor_d435> -->
+        <joint name="base_joint" type="fixed">
+            <origin rpy="0 0 0" xyz="0 0 0" />
+            <parent link="world" />
+            <child link="base_link" />
+        </joint>
         <!-- <link name="camera_link">
         <visual>
@@ -59,9 +69,4 @@
         <child link="camera_link" />
     </joint> -->
-        <joint name="world_to_base" type="fixed">
-            <xacro:insert_block name="origin" />
-            <parent link="${parent}" />
-            <child link="base_link" />
-        </joint>
         <link name="base_link" />
         <joint name="base_link-base_link_inertia" type="fixed">
@@ -359,4 +364,63 @@
         </inertial>
     </link> -->
+        <ros2_control name="URBot" type="system">
+            <hardware>
+                <plugin>gazebo_ros2_control/GazeboSystem</plugin>
+            </hardware>
+            <joint name="shoulder_pan_joint">
+                <command_interface name="position">
+                    <param name="min">{-2*pi}</param>
+                    <param name="max">{2*pi}</param>
+                </command_interface>
+                <state_interface name="position">
+                    <param name="initial_value">0.0</param>
+                </state_interface>
+            </joint>
+            <joint name="shoulder_lift_joint">
+                <command_interface name="position">
+                    <param name="min">{-2*pi}</param>
+                    <param name="max">{2*pi}</param>
+                </command_interface>
+                <state_interface name="position">
+                    <param name="initial_value">0</param>
+                </state_interface>
+            </joint>
+            <joint name="elbow_joint">
+                <command_interface name="position">
+                    <param name="min">{-pi}</param>
+                    <param name="max">{pi}</param>
+                </command_interface>
+                <state_interface name="position">
+                    <param name="initial_value">0.0</param>
+                </state_interface>
+            </joint>
+            <joint name="wrist_1_joint">
+                <command_interface name="position">
+                    <param name="min">{-2*pi}</param>
+                    <param name="max">{2*pi}</param>
+                </command_interface>
+                <state_interface name="position">
+                    <param name="initial_value">0</param>
+                </state_interface>
+            </joint>
+            <joint name="wrist_2_joint">
+                <command_interface name="position">
+                    <param name="min">{-2*pi}</param>
+                    <param name="max">{2*pi}</param>
+                </command_interface>
+                <state_interface name="position">
+                    <param name="initial_value">0</param>
+                </state_interface>
+            </joint>
+            <joint name="wrist_3_joint">
+                <command_interface name="position">
+                    <param name="min">{-2*pi}</param>
+                    <param name="max">{2*pi}</param>
+                </command_interface>
+                <state_interface name="position">
+                    <param name="initial_value">0</param>
+                </state_interface>
+            </joint>
+        </ros2_control>
         <!-- Link1 -->
         <gazebo reference="base_link_inertia">

File: gazebo_env/description/urdf/ur5e_with_gripper.urdf.xacro (robot description, xacro)
@@ -4,12 +4,7 @@
     <xacro:include filename="$(find gazebo_env)/urdf/ur5e.urdf.xacro" />
     <xacro:include filename="$(find robotiq_description)/urdf/ur_to_robotiq_adapter.urdf.xacro" />
-    <link name="world" />
-    <xacro:ur5e parent="world">
-        <origin xyz="0 0 0" rpy="0 0 0" />
-    </xacro:ur5e>
+    <xacro:ur5e />
     <xacro:ur_to_robotiq prefix="" connected_to="tool0"/>
-    <!-- parameters -->
     <xacro:arg name="use_fake_hardware" default="true" />
-    <!-- Import macros -->
     <xacro:include filename="$(find robotiq_description)/urdf/robotiq_2f_85_macro.urdf.xacro" />
     <xacro:robotiq_gripper name="RobotiqGripperHardwareInterface" prefix="" parent="gripper_mount_link" use_fake_hardware="$(arg use_fake_hardware)">

File: robotiq_description/urdf/robotiq_2f_85_macro.urdf.xacro (robot description, xacro)
@@ -5,22 +5,10 @@
         prefix
         parent
-        *origin
-        sim_ignition:=false
-        sim_isaac:=false
-        use_fake_hardware:=false
-        fake_sensor_commands:=false
-        include_ros2_control:=true
-        com_port:=/dev/ttyUSB0">
+        *origin sim_ignition:=false sim_isaac:=false use_fake_hardware:=false fake_sensor_commands:=false include_ros2_control:=true com_port:=/dev/ttyUSB0">
         <!-- ros2 control include -->
         <xacro:include filename="$(find robotiq_description)/urdf/robotiq_gripper.ros2_control.xacro" />
         <!-- if we are simulating or directly communicating with the gripper we need a ros2 control instance -->
         <xacro:if value="${include_ros2_control}">
-            <xacro:robotiq_gripper_ros2_control
-                name="${name}" prefix="${prefix}"
-                sim_ignition="${sim_ignition}"
-                sim_isaac="${sim_isaac}"
-                use_fake_hardware="${use_fake_hardware}"
-                fake_sensor_commands="${fake_sensor_commands}"
-                com_port="${com_port}"/>
+            <xacro:robotiq_gripper_ros2_control name="${name}" prefix="${prefix}" sim_ignition="${sim_ignition}" sim_isaac="${sim_isaac}" use_fake_hardware="${use_fake_hardware}" fake_sensor_commands="${fake_sensor_commands}" com_port="${com_port}"/>
         </xacro:if>
         <link name="${prefix}robotiq_85_base_link">
@@ -155,18 +143,18 @@
                 <surface>
                     <friction>
-                    <ode>
-                        <mu1>100000.0</mu1>
-                        <mu2>100000.0</mu2>
-                    </ode>
+                        <ode>
+                            <mu1>100000.0</mu1>
+                            <mu2>100000.0</mu2>
+                        </ode>
                     </friction>
                     <contact>
-                    <ode>
-                        <kp>1e+5</kp>
-                        <kd>1</kd>
-                        <soft_cfm>0</soft_cfm>
-                        <soft_erp>0.2</soft_erp>
-                        <minDepth>0.002</minDepth>
-                        <maxVel>0</maxVel>
-                    </ode>
+                        <ode>
+                            <kp>1e+5</kp>
+                            <kd>1</kd>
+                            <soft_cfm>0</soft_cfm>
+                            <soft_erp>0.2</soft_erp>
+                            <minDepth>0.002</minDepth>
+                            <maxVel>0</maxVel>
+                        </ode>
                     </contact>
                 </surface>
@@ -190,18 +178,18 @@
                 <surface>
                     <friction>
-                    <ode>
-                        <mu1>100000.0</mu1>
-                        <mu2>100000.0</mu2>
-                    </ode>
+                        <ode>
+                            <mu1>100000.0</mu1>
+                            <mu2>100000.0</mu2>
+                        </ode>
                     </friction>
                     <contact>
-                    <ode>
-                        <kp>1e+5</kp>
-                        <kd>1</kd>
-                        <soft_cfm>0</soft_cfm>
-                        <soft_erp>0.2</soft_erp>
-                        <minDepth>0.002</minDepth>
-                        <maxVel>0</maxVel>
-                    </ode>
+                        <ode>
+                            <kp>1e+5</kp>
+                            <kd>1</kd>
+                            <soft_cfm>0</soft_cfm>
+                            <soft_erp>0.2</soft_erp>
+                            <minDepth>0.002</minDepth>
+                            <maxVel>0</maxVel>
+                        </ode>
                     </contact>
                 </surface>
@@ -212,4 +200,16 @@
                 <inertia ixx="1.048152e-05" iyy="1.197888e-05" izz="4.22784e-06" ixy="0.0" ixz="-3.5232e-06" iyz="0.0" />
             </inertial>
+        </link>
+        <link name ="true_end_effector">
+            <!-- <visual>
+                <geometry>
+                    <sphere radius="0.01"/>
+                </geometry>
+            </visual>
+            <inertial>
+                <origin xyz="0 0 0" rpy="0 0 0" />
+                <mass value="4.268588744e-02" />
+                <inertia ixx="1.048152e-05" iyy="1.197888e-05" izz="4.22784e-06" ixy="0.0" ixz="-3.5232e-06" iyz="0.0" />
+            </inertial> -->
         </link>
         <joint name="${prefix}robotiq_85_base_joint" type="fixed">
@@ -225,4 +225,9 @@
             <limit lower="0.0" upper="0.8" velocity="0.5" effort="50" />
         </joint>
+        <joint name="dummy_ee_joint" type="fixed">
+            <parent link="${prefix}robotiq_85_base_link" />
+            <child link="true_end_effector" />
+            <origin xyz="0.0 0.0 0.098" rpy="0 0 0" />
+        </joint>
         <joint name="${prefix}robotiq_85_right_knuckle_joint" type="revolute">
             <parent link="${prefix}robotiq_85_base_link" />
