Commit message: Run gazebo classic and the pointcloud publisher, and we have pointcloud for the robot

File: gazebo_env/description/urdf/ur5e_gazebo_pointcloud_debug.urdf.xacro (robot description, xacro)
@@ -46,27 +46,6 @@
         <origin rpy="0 0 0" xyz="0 0 0" />
         <parent link="world" />
-        <child link="forearm_link" />
-    </joint>
-    <!-- <link name="camera_link">
-        <visual>
-            <origin xyz="0 0 0" rpy="0 0 0" />
-            <geometry>
-                <box size="0.09 0.025 0.025" />
-            </geometry>
-        </visual>
-        <inertial>
-            <origin xyz="0 0 0" rpy="0 0 0" />
-            <mass value="1" />
-            <inertia
-                ixx="1.0" ixy="0.0" ixz="0.0"
-                iyy="1.0" iyz="0.0"
-                izz="1.0" />
-        </inertial>
-    </link>
-    <joint name="camera_joint" type="fixed">
-        <origin rpy="0 0 2.35619449" xyz="1 1 0.0125" />
-        <parent link="world" />
-        <child link="camera_link" />
-    </joint> -->
+        <child link="wrist_1_link" />
+    </joint>
     <!-- <link name="base_link" />
     <joint name="base_link-base_link_inertia" type="fixed">
@@ -107,6 +86,6 @@
             soft_upper_limit="6.133185307179586" />
         <dynamics damping="0" friction="0" />
-    </joint>
-    <link name="shoulder_link">
+    </joint> -->
+    <!-- <link name="shoulder_link">
         <visual>
             <origin rpy="0 0 3.141592653589793" xyz="0 0 0" />
@@ -129,6 +108,6 @@
                 izz="0.00666" />
         </inertial>
-    </link>
-    <joint name="shoulder_lift_joint" type="revolute">
+    </link> -->
+    <!-- <joint name="shoulder_lift_joint" type="revolute">
         <parent link="shoulder_link" />
         <child link="upper_arm_link" />
@@ -140,6 +119,6 @@
             soft_upper_limit="6.133185307179586" />
         <dynamics damping="0" friction="0" />
-    </joint>
-    <link name="upper_arm_link">
+    </joint> -->
+    <!-- <link name="upper_arm_link">
         <visual>
             <origin rpy="1.5707963267948966 0 -1.5707963267948966" xyz="0 0 0.138" />
@@ -162,6 +141,6 @@
                 izz="0.0151074" />
         </inertial>
-    </link>
-    <joint name="elbow_joint" type="revolute">
+    </link> -->
+    <!-- <joint name="elbow_joint" type="revolute">
         <parent link="upper_arm_link" />
         <child link="forearm_link" />
@@ -174,5 +153,5 @@
         <dynamics damping="0" friction="0" />
     </joint> -->
-    <link name="forearm_link">
+    <!-- <link name="forearm_link">
         <visual>
             <origin rpy="1.5707963267948966 0 -1.5707963267948966" xyz="0 0 0.007" />
@@ -196,5 +175,5 @@
                 izz="0.004095" />
         </inertial>
-    </link>
+    </link> -->
     <!-- <joint name="wrist_1_joint" type="revolute">
         <parent link="forearm_link" />
@@ -207,5 +186,5 @@
             soft_upper_limit="6.133185307179586" />
         <dynamics damping="0" friction="0" />
-    </joint>
+    </joint> -->
     <link name="wrist_1_link">
         <visual>
@@ -231,5 +210,5 @@
         </inertial>
     </link>
-    <joint name="wrist_2_joint" type="revolute">
+    <!-- <joint name="wrist_2_joint" type="revolute">
         <parent link="wrist_1_link" />
         <child link="wrist_2_link" />
