Commit message: Temp commit

File: gazebo_env/description/urdf/ur5e_gazebo.urdf.xacro (robot description, xacro)
@@ -11,5 +11,5 @@
 -->
 <robot name="2dof_robot" xmlns:xacro="http://ros.org/wiki/xacro">
-    <xacro:include filename="$(find gazebo_env)/urdf/d435.urdf.xacro" />
+    <!-- <xacro:include filename="$(find gazebo_env)/urdf/d435.urdf.xacro" />
     <material name="black">
         <color rgba="0.0 0.0 0.0 1.0" />
@@ -38,10 +38,9 @@
     <material name="white">
         <color rgba="1.0 1.0 1.0 1.0" />
-    </material>
-    <!-- Used for fixing robot -->
+    </material> -->
     <link name="world" />
-    <xacro:sensor_d435 parent="world">
+    <!-- <xacro:sensor_d435 parent="world">
         <origin xyz="1.5 1.5 1" rpy="0 0.5235987756 -2.35619449" />
-    </xacro:sensor_d435>
+    </xacro:sensor_d435> -->
     <joint name="base_joint" type="fixed">
         <origin rpy="0 0 0" xyz="0 0 0" />
@@ -476,5 +475,5 @@
         <plugin filename="libgazebo_ros2_control.so" name="gazebo_ros2_control">
             <parameters>
-                /home/kushtimusprime/cross_embodiment_test_ws/install/gazebo_env/share/gazebo_env/config/urbot_controllers.yaml
+                /home/benchturtle/cross_embodiment_ws/src/gazebo_env/bringup/config/urbot_controllers.yaml
             </parameters>
         </plugin>

Commit message: Now, if you run gazebo classic launch and the pointcloud publisher, you will get segmentation masks of the robot

File: gazebo_env/description/urdf/ur5e_gazebo.urdf.xacro (robot description, xacro)
@@ -10,6 +10,8 @@
 https://github.com/ros-simulation/gazebo_ros_demos/blob/kinetic-devel/rrbot_description/urdf/rrbot.xacro
 -->
-<robot name="2dof_robot" xmlns:xacro="http://ros.org/wiki/xacro">
-    <!-- <xacro:include filename="$(find gazebo_env)/urdf/d435.urdf.xacro" />
+<robot name="ur5e" xmlns:xacro="http://ros.org/wiki/xacro">
+    <xacro:macro name="ur5e"
+        params="parent:=world *origin name:=ur5e">
+        <!-- <xacro:include filename="$(find gazebo_env)/urdf/d435.urdf.xacro" />
     <material name="black">
         <color rgba="0.0 0.0 0.0 1.0" />
@@ -39,14 +41,13 @@
         <color rgba="1.0 1.0 1.0 1.0" />
     </material> -->
-    <link name="world" />
-    <!-- <xacro:sensor_d435 parent="world">
+        <!-- <xacro:sensor_d435 parent="world">
         <origin xyz="1.5 1.5 1" rpy="0 0.5235987756 -2.35619449" />
     </xacro:sensor_d435> -->
-    <joint name="base_joint" type="fixed">
-        <origin rpy="0 0 0" xyz="0 0 0" />
-        <parent link="world" />
-        <child link="base_link" />
-    </joint>
-    <!-- <link name="camera_link">
+        <joint name="base_joint" type="fixed">
+            <xacro:insert_block name="origin" />
+            <parent link="${parent}" />
+            <child link="base_link" />
+        </joint>
+        <!-- <link name="camera_link">
         <visual>
             <origin xyz="0 0 0" rpy="0 0 0" />
@@ -69,262 +70,269 @@
         <child link="camera_link" />
     </joint> -->
-    <link name="base_link" />
-    <joint name="base_link-base_link_inertia" type="fixed">
-        <parent link="base_link" />
-        <child link="base_link_inertia" />
-        <!-- 'base_link' is REP-103 aligned (so X+ forward), while the internal
+        <link name="base_link" />
+        <joint name="base_link-base_link_inertia" type="fixed">
+            <parent link="base_link" />
+            <child link="base_link_inertia" />
+            <!-- 'base_link' is REP-103 aligned (so X+ forward), while the internal
                frames of the robot/controller have X+ pointing backwards.
                Use the joint between 'base_link' and 'base_link_inertia' (a dummy
                link/frame) to introduce the necessary rotation over Z (of pi rad).
           -->
-        <origin rpy="0 0 3.141592653589793" xyz="0 0 0" />
-    </joint>
-    <link name="base_link_inertia">
-        <collision>
             <origin rpy="0 0 3.141592653589793" xyz="0 0 0" />
-            <geometry>
-                <mesh
-                    filename="file://$(find gazebo_env)/meshes/ur5e/collision/base.stl" />
-            </geometry>
-        </collision>
-        <visual>
-            <origin rpy="0 0 3.141592653589793" xyz="0 0 0" />
-            <geometry>
-                <mesh
-                    filename="file://$(find gazebo_env)/meshes/ur5e/visual/base.dae" />
-            </geometry>
-        </visual>
-        <inertial>
-            <mass value="4.0" />
-            <origin rpy="0 0 0" xyz="0 0 0" />
-            <inertia ixx="0.00443333156" ixy="0.0" ixz="0.0" iyy="0.00443333156" iyz="0.0"
-                izz="0.0072" />
-        </inertial>
-    </link>
-    <joint name="shoulder_pan_joint" type="revolute">
-        <parent link="base_link_inertia" />
-        <child link="shoulder_link" />
-        <origin rpy="0 0 0" xyz="0 0 0.1625" />
-        <axis xyz="0 0 1" />
-        <limit effort="150.0" lower="-6.283185307179586" upper="6.283185307179586"
-            velocity="3.141592653589793" />
-        <safety_controller k_position="20" k_velocity="0.0" soft_lower_limit="-6.133185307179586"
-            soft_upper_limit="6.133185307179586" />
-        <dynamics damping="0" friction="0" />
-    </joint>
-    <link name="shoulder_link">
-        <visual>
-            <origin rpy="0 0 3.141592653589793" xyz="0 0 0" />
-            <geometry>
-                <mesh
-                    filename="file://$(find gazebo_env)/meshes/ur5e/visual/shoulder.dae" />
-            </geometry>
-        </visual>
-        <collision>
-            <origin rpy="0 0 3.141592653589793" xyz="0 0 0" />
-            <geometry>
-                <mesh
-                    filename="file://$(find gazebo_env)/meshes/ur5e/collision/shoulder.stl" />
-            </geometry>
-        </collision>
-        <inertial>
-            <mass value="3.7" />
-            <origin rpy="0 0 0" xyz="0 0 0" />
-            <inertia ixx="0.010267495893" ixy="0.0" ixz="0.0" iyy="0.010267495893" iyz="0.0"
-                izz="0.00666" />
-        </inertial>
-    </link>
-    <joint name="shoulder_lift_joint" type="revolute">
-        <parent link="shoulder_link" />
-        <child link="upper_arm_link" />
-        <origin rpy="1.570796327 0 0" xyz="0 0 0" />
-        <axis xyz="0 0 1" />
-        <limit effort="150.0" lower="-6.283185307179586" upper="6.283185307179586"
-            velocity="3.141592653589793" />
-        <safety_controller k_position="20" k_velocity="0.0" soft_lower_limit="-6.133185307179586"
-            soft_upper_limit="6.133185307179586" />
-        <dynamics damping="0" friction="0" />
-    </joint>
-    <link name="upper_arm_link">
-        <visual>
-            <origin rpy="1.5707963267948966 0 -1.5707963267948966" xyz="0 0 0.138" />
-            <geometry>
-                <mesh
-                    filename="file://$(find gazebo_env)/meshes/ur5e/visual/upperarm.dae" />
-            </geometry>
-        </visual>
-        <collision>
-            <origin rpy="1.5707963267948966 0 -1.5707963267948966" xyz="0 0 0.138" />
-            <geometry>
-                <mesh
-                    filename="file://$(find gazebo_env)/meshes/ur5e/collision/upperarm.stl" />
-            </geometry>
-        </collision>
-        <inertial>
-            <mass value="0.8393" />
-            <origin rpy="0 1.5707963267948966 0" xyz="-0.2125 0.0 0.138" />
-            <inertia ixx="0.1338857818623325" ixy="0.0" ixz="0.0" iyy="0.1338857818623325" iyz="0.0"
-                izz="0.0151074" />
-        </inertial>
-    </link>
-    <joint name="elbow_joint" type="revolute">
-        <parent link="upper_arm_link" />
-        <child link="forearm_link" />
-        <origin rpy="0 0 0" xyz="-0.425 0 0" />
-        <axis xyz="0 0 1" />
-        <limit effort="150.0" lower="-3.141592653589793" upper="3.141592653589793"
-            velocity="3.141592653589793" />
-        <safety_controller k_position="20" k_velocity="0.0" soft_lower_limit="-2.991592653589793"
-            soft_upper_limit="2.991592653589793" />
-        <dynamics damping="0" friction="0" />
-    </joint>
-    <link name="forearm_link">
-        <visual>
-            <origin rpy="1.5707963267948966 0 -1.5707963267948966" xyz="0 0 0.007" />
-            <geometry>
-                <mesh
-                    filename="file://$(find gazebo_env)/meshes/ur5e/visual/forearm.dae" />
-            </geometry>
-        </visual>
-        <collision>
-            <origin rpy="1.5707963267948966 0 -1.5707963267948966" xyz="0 0 0.007" />
-            <geometry>
-                <mesh
-                    filename="file://$(find gazebo_env)/meshes/ur5e/collision/forearm.stl" />
-            </geometry>
-        </collision>
-        <inertial>
-            <mass value="2.275" />
-            <origin rpy="0 1.5707963267948966 0" xyz="-0.1961 0.0 0.007" />
-            <inertia ixx="0.031209355099586295" ixy="0.0" ixz="0.0" iyy="0.031209355099586295"
-                iyz="0.0"
-                izz="0.004095" />
-        </inertial>
-    </link>
-    <joint name="wrist_1_joint" type="revolute">
-        <parent link="forearm_link" />
-        <child link="wrist_1_link" />
-        <origin rpy="0 0 0" xyz="-0.3922 0 0.1333" />
-        <axis xyz="0 0 1" />
-        <limit effort="28.0" lower="-6.283185307179586" upper="6.283185307179586"
-            velocity="3.141592653589793" />
-        <safety_controller k_position="20" k_velocity="0.0" soft_lower_limit="-6.133185307179586"
-            soft_upper_limit="6.133185307179586" />
-        <dynamics damping="0" friction="0" />
-    </joint>
-    <link name="wrist_1_link">
-        <visual>
-            <origin rpy="1.5707963267948966 0 0" xyz="0 0 -0.127" />
-            <geometry>
-                <mesh
-                    filename="file://$(find gazebo_env)/meshes/ur5e/visual/wrist1.dae" />
-            </geometry>
-        </visual>
-        <collision>
-            <origin rpy="1.5707963267948966 0 0" xyz="0 0 -0.127" />
-            <geometry>
-                <mesh
-                    filename="file://$(find gazebo_env)/meshes/ur5e/collision/wrist1.stl" />
-            </geometry>
-        </collision>
-        <inertial>
-            <mass value="1.219" />
-            <origin rpy="0 0 0" xyz="0 0 0" />
-            <inertia ixx="0.0025598989760400002" ixy="0.0" ixz="0.0" iyy="0.0025598989760400002"
-                iyz="0.0"
-                izz="0.0021942" />
-        </inertial>
-    </link>
-    <joint name="wrist_2_joint" type="revolute">
-        <parent link="wrist_1_link" />
-        <child link="wrist_2_link" />
-        <origin rpy="1.570796327 0 0" xyz="0 -0.0997 -2.044881182297852e-11" />
-        <axis xyz="0 0 1" />
-        <limit effort="28.0" lower="-6.283185307179586" upper="6.283185307179586"
-            velocity="3.141592653589793" />
-        <safety_controller k_position="20" k_velocity="0.0" soft_lower_limit="-6.133185307179586"
-            soft_upper_limit="6.133185307179586" />
-        <dynamics damping="0" friction="0" />
-    </joint>
-    <link name="wrist_2_link">
-        <visual>
-            <origin rpy="0 0 0" xyz="0 0 -0.0997" />
-            <geometry>
-                <mesh
-                    filename="file://$(find gazebo_env)/meshes/ur5e/visual/wrist2.dae" />
-            </geometry>
-        </visual>
-        <collision>
-            <origin rpy="0 0 0" xyz="0 0 -0.0997" />
-            <geometry>
-                <mesh
-                    filename="file://$(find gazebo_env)/meshes/ur5e/collision/wrist2.stl" />
-            </geometry>
-        </collision>
-        <inertial>
-            <mass value="1.219" />
-            <origin rpy="0 0 0" xyz="0 0 0" />
-            <inertia ixx="0.0025598989760400002" ixy="0.0" ixz="0.0" iyy="0.0025598989760400002"
-                iyz="0.0"
-                izz="0.0021942" />
-        </inertial>
-    </link>
-    <joint name="wrist_3_joint" type="revolute">
-        <parent link="wrist_2_link" />
-        <child link="wrist_3_link" />
-        <origin rpy="1.570796326589793 3.141592653589793 3.141592653589793"
-            xyz="0 0.0996 -2.042830148012698e-11" />
-        <axis xyz="0 0 1" />
-        <limit effort="28.0" lower="-6.283185307179586" upper="6.283185307179586"
-            velocity="3.141592653589793" />
-        <safety_controller k_position="20" k_velocity="0.0" soft_lower_limit="-6.133185307179586"
-            soft_upper_limit="6.133185307179586" />
-        <dynamics damping="0" friction="0" />
-    </joint>
-    <link name="wrist_3_link">
-        <visual>
-            <origin rpy="1.5707963267948966 0 0" xyz="0 0 -0.0989" />
-            <geometry>
-                <mesh
-                    filename="file://$(find gazebo_env)/meshes/ur5e/visual/wrist3.dae" />
-            </geometry>
-        </visual>
-        <collision>
-            <origin rpy="1.5707963267948966 0 0" xyz="0 0 -0.0989" />
-            <geometry>
-                <mesh
-                    filename="file://$(find gazebo_env)/meshes/ur5e/collision/wrist3.stl" />
-            </geometry>
-        </collision>
-        <inertial>
-            <mass value="0.1879" />
-            <origin rpy="0 0 0" xyz="0.0 0.0 -0.0229" />
-            <inertia ixx="9.890410052167731e-05" ixy="0.0" ixz="0.0" iyy="9.890410052167731e-05"
-                iyz="0.0"
-                izz="0.0001321171875" />
-        </inertial>
-    </link>
-    <link name="ft_frame" />
-    <joint name="wrist_3_link-ft_frame" type="fixed">
-        <parent link="wrist_3_link" />
-        <child link="ft_frame" />
-        <origin rpy="3.141592653589793 0 0" xyz="0 0 0" />
-    </joint>
-    <link name="flange" />
-    <joint name="wrist_3-flange" type="fixed">
-        <parent link="wrist_3_link" />
-        <child link="flange" />
-        <origin rpy="0 -1.5707963267948966 -1.5707963267948966" xyz="0 0 0" />
-    </joint>
-    <!-- ROS-Industrial 'tool0' frame - all-zeros tool frame -->
-    <link name="tool0" />
-    <joint name="flange-tool0" type="fixed">
-        <!-- default toolframe - X+ left, Y+ up, Z+ front -->
-        <origin rpy="1.5707963267948966 0 1.5707963267948966" xyz="0 0 0" />
-        <parent link="flange" />
-        <child link="tool0" />
-    </joint>
-    <!-- Base Link -->
-    <!-- <link name="base_link">
+        </joint>
+        <link name="base_link_inertia">
+            <collision>
+                <origin rpy="0 0 3.141592653589793" xyz="0 0 0" />
+                <geometry>
+                    <mesh
+                        filename="file://$(find gazebo_env)/meshes/ur5e/collision/base.stl" />
+                </geometry>
+            </collision>
+            <visual>
+                <origin rpy="0 0 3.141592653589793" xyz="0 0 0" />
+                <geometry>
+                    <mesh
+                        filename="file://$(find gazebo_env)/meshes/ur5e/visual/base.dae" />
+                </geometry>
+            </visual>
+            <inertial>
+                <mass value="4.0" />
+                <origin rpy="0 0 0" xyz="0 0 0" />
+                <inertia ixx="0.00443333156" ixy="0.0" ixz="0.0" iyy="0.00443333156" iyz="0.0"
+                    izz="0.0072" />
+            </inertial>
+        </link>
+        <joint name="shoulder_pan_joint" type="revolute">
+            <parent link="base_link_inertia" />
+            <child link="shoulder_link" />
+            <origin rpy="0 0 0" xyz="0 0 0.1625" />
+            <axis xyz="0 0 1" />
+            <limit effort="150.0" lower="-6.283185307179586" upper="6.283185307179586"
+                velocity="3.141592653589793" />
+            <safety_controller k_position="20" k_velocity="0.0"
+                soft_lower_limit="-6.133185307179586"
+                soft_upper_limit="6.133185307179586" />
+            <dynamics damping="0" friction="0" />
+        </joint>
+        <link name="shoulder_link">
+            <visual>
+                <origin rpy="0 0 3.141592653589793" xyz="0 0 0" />
+                <geometry>
+                    <mesh
+                        filename="file://$(find gazebo_env)/meshes/ur5e/visual/shoulder.dae" />
+                </geometry>
+            </visual>
+            <collision>
+                <origin rpy="0 0 3.141592653589793" xyz="0 0 0" />
+                <geometry>
+                    <mesh
+                        filename="file://$(find gazebo_env)/meshes/ur5e/collision/shoulder.stl" />
+                </geometry>
+            </collision>
+            <inertial>
+                <mass value="3.7" />
+                <origin rpy="0 0 0" xyz="0 0 0" />
+                <inertia ixx="0.010267495893" ixy="0.0" ixz="0.0" iyy="0.010267495893" iyz="0.0"
+                    izz="0.00666" />
+            </inertial>
+        </link>
+        <joint name="shoulder_lift_joint" type="revolute">
+            <parent link="shoulder_link" />
+            <child link="upper_arm_link" />
+            <origin rpy="1.570796327 0 0" xyz="0 0 0" />
+            <axis xyz="0 0 1" />
+            <limit effort="150.0" lower="-6.283185307179586" upper="6.283185307179586"
+                velocity="3.141592653589793" />
+            <safety_controller k_position="20" k_velocity="0.0"
+                soft_lower_limit="-6.133185307179586"
+                soft_upper_limit="6.133185307179586" />
+            <dynamics damping="0" friction="0" />
+        </joint>
+        <link name="upper_arm_link">
+            <visual>
+                <origin rpy="1.5707963267948966 0 -1.5707963267948966" xyz="0 0 0.138" />
+                <geometry>
+                    <mesh
+                        filename="file://$(find gazebo_env)/meshes/ur5e/visual/upperarm.dae" />
+                </geometry>
+            </visual>
+            <collision>
+                <origin rpy="1.5707963267948966 0 -1.5707963267948966" xyz="0 0 0.138" />
+                <geometry>
+                    <mesh
+                        filename="file://$(find gazebo_env)/meshes/ur5e/collision/upperarm.stl" />
+                </geometry>
+            </collision>
+            <inertial>
+                <mass value="0.8393" />
+                <origin rpy="0 1.5707963267948966 0" xyz="-0.2125 0.0 0.138" />
+                <inertia ixx="0.1338857818623325" ixy="0.0" ixz="0.0" iyy="0.1338857818623325"
+                    iyz="0.0"
+                    izz="0.0151074" />
+            </inertial>
+        </link>
+        <joint name="elbow_joint" type="revolute">
+            <parent link="upper_arm_link" />
+            <child link="forearm_link" />
+            <origin rpy="0 0 0" xyz="-0.425 0 0" />
+            <axis xyz="0 0 1" />
+            <limit effort="150.0" lower="-3.141592653589793" upper="3.141592653589793"
+                velocity="3.141592653589793" />
+            <safety_controller k_position="20" k_velocity="0.0"
+                soft_lower_limit="-2.991592653589793"
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