Commit message: Temp commit

File: gazebo_env/description/urdf/ur5e_camera_gazebo_scene.urdf.xacro (robot description, xacro)
@@ -18,5 +18,6 @@
     </xacro:ur5e>
     <xacro:sensor_d435 parent="world">
-        <origin xyz="1.5 1.5 1" rpy="0 0.5235987756 -2.35619449" />
+        <origin xyz="1.5 1.5 1" rpy="0 0.4405106 -2.3561945" />
+        <!-- <origin xyz="-1 0 0" rpy="0 3.1415927 1.5707963" /> -->
     </xacro:sensor_d435>
 </robot>

Commit message: We have added the gripper

File: gazebo_env/description/urdf/ur5e_camera_gazebo_scene.urdf.xacro (robot description, xacro)
@@ -13,8 +13,15 @@
     <xacro:include filename="$(find gazebo_env)/urdf/ur5e_gazebo.urdf.xacro" />
     <xacro:include filename="$(find gazebo_env)/urdf/d435.urdf.xacro" />
+    <xacro:include filename="$(find robotiq_description)/urdf/ur_to_robotiq_adapter.urdf.xacro" />
     <link name="world" />
     <xacro:ur5e parent="world">
         <origin xyz="0 0 0" rpy="0 0 0" />
     </xacro:ur5e>
+    <xacro:ur_to_robotiq prefix="" connected_to="tool0"/>
+    <xacro:arg name="use_fake_hardware" default="true" />
+    <xacro:include filename="$(find robotiq_description)/urdf/robotiq_2f_85_macro.urdf.xacro" />
+    <xacro:robotiq_gripper prefix="" parent="gripper_mount_link">
+        <origin xyz="0 0 0" rpy="0 0 0" />
+    </xacro:robotiq_gripper>
     <xacro:sensor_d435 parent="world">
         <origin xyz="1.5 1.5 1" rpy="0 0.4405106 -2.3561945" />

File: gazebo_env/description/urdf/ur5e_with_gripper.urdf.xacro (robot description, xacro)
@@ -1,23 +1,25 @@
 <?xml version="1.0"?>
-<robot name="ur5e_with_gripper"
-    xmlns:xacro="http://ros.org/wiki/xacro">
-    <xacro:include filename="$(find gazebo_env)/urdf/ur5e.urdf.xacro" />
+<!-- =================================================================================== -->
+<!-- |    This document was autogenerated by xacro from
+install/share/gazebo_env/urdf/rrbot.urdf.xacro | -->
+<!-- |    EDITING THIS FILE BY HAND IS NOT RECOMMENDED                                 | -->
+<!-- =================================================================================== -->
+<!-- Revolute-Revolute Manipulator -->
+<!--
+Copied and modified from ROS1 example -
+https://github.com/ros-simulation/gazebo_ros_demos/blob/kinetic-devel/rrbot_description/urdf/rrbot.xacro
+-->
+<robot name="ur5e_scene" xmlns:xacro="http://ros.org/wiki/xacro">
+    <xacro:include filename="$(find gazebo_env)/urdf/ur5e_gazebo.urdf.xacro" />
     <xacro:include filename="$(find robotiq_description)/urdf/ur_to_robotiq_adapter.urdf.xacro" />
-    <xacro:ur5e />
+    <link name="world" />
+    <xacro:ur5e parent="world">
+        <origin xyz="0 0 0" rpy="0 0 0" />
+    </xacro:ur5e>
     <xacro:ur_to_robotiq prefix="" connected_to="tool0"/>
     <xacro:arg name="use_fake_hardware" default="true" />
     <xacro:include filename="$(find robotiq_description)/urdf/robotiq_2f_85_macro.urdf.xacro" />
-    <xacro:robotiq_gripper name="RobotiqGripperHardwareInterface" prefix="" parent="gripper_mount_link" use_fake_hardware="$(arg use_fake_hardware)">
+    <xacro:robotiq_gripper prefix="" parent="gripper_mount_link">
         <origin xyz="0 0 0" rpy="0 0 0" />
     </xacro:robotiq_gripper>
-    <gazebo>
-        <plugin filename="libgazebo_ros2_control.so" name="gazebo_ros2_control">
-            <parameters>
-                /home/kushtimusprime/cross_embodiment_test_ws/src/robotiq_driver/config/basic_controller.yaml
-            </parameters>
-        </plugin>
-    </gazebo>
-    <gazebo>
-        <plugin name="control" filename="libcontrol_plugin.so" />
-    </gazebo>
 </robot>
