Commit message: Temp update

File: gazebo_env/description/urdf/ur5e_with_gripper_gazebo_solo.urdf.xacro (robot description, xacro)
@@ -12,13 +12,15 @@
 <robot name="ur5e_scene" xmlns:xacro="http://ros.org/wiki/xacro">
     <xacro:include filename="$(find gazebo_env)/urdf/ur5e_gazebo.urdf.xacro" />
+    <xacro:include filename="$(find gazebo_env)/urdf/d435.urdf.xacro" />
     <xacro:include filename="$(find robotiq_description)/urdf/ur_to_robotiq_adapter.urdf.xacro" />
+    <xacro:include filename="$(find robotiq_description)/urdf/robotiq_2f_85_macro.urdf.xacro" />
     <link name="world" />
-    <xacro:ur5e parent="world">
+    <!-- <xacro:ur5e parent="world">
         <origin xyz="0 0 0" rpy="0 0 0" />
-    </xacro:ur5e>
-    <xacro:ur_to_robotiq prefix="" connected_to="tool0"/>
-    <xacro:arg name="use_fake_hardware" default="true" />
+    </xacro:ur5e> -->
+    <!-- <xacro:ur_to_robotiq prefix="" connected_to="world"/>
+    <xacro:arg name="use_fake_hardware" default="true" /> -->
     <xacro:include filename="$(find robotiq_description)/urdf/robotiq_2f_85_macro.urdf.xacro" />
-    <xacro:robotiq_gripper prefix="" parent="gripper_mount_link">
+    <xacro:robotiq_gripper prefix="" parent="world">
         <origin xyz="0 0 0" rpy="0 0 0" />
     </xacro:robotiq_gripper>

File: robotiq_description/urdf/robotiq_2f_85_macro.urdf.xacro (robot description, xacro)
@@ -39,10 +39,15 @@
             <parent link="${prefix}robotiq_85_base_link" />
             <child link="${prefix}robotiq_85_left_knuckle_link" />
-            <axis xyz="0 -1 0" />
             <origin xyz="0.03060114 0.0 0.05490452" rpy="0 0 0" />
+            <axis xyz="0 -1 0" />
             <limit lower="0.0" upper="0.8" velocity="0.5" effort="50" />
+            <safety_controller k_position="20" k_velocity="0.0"
+                soft_lower_limit="-6.133185307179586"
+                soft_upper_limit="6.133185307179586" />
+            <dynamics damping="0" friction="0" />
         </joint>
         <link name="${prefix}robotiq_85_left_knuckle_link">
             <visual>
+                <origin rpy="0 0 0" xyz="0 0 0"/>
                 <geometry>
                     <mesh
@@ -65,4 +70,5 @@
         <link name="${prefix}robotiq_85_right_knuckle_link">
             <visual>
+                <origin rpy="0 0 0" xyz="0 0 0"/>
                 <geometry>
                     <mesh
@@ -85,4 +91,5 @@
         <link name="${prefix}robotiq_85_left_finger_link">
             <visual>
+                <origin rpy="0 0 0" xyz="0 0 0"/>
                 <geometry>
                     <mesh
@@ -105,4 +112,5 @@
         <link name="${prefix}robotiq_85_right_finger_link">
             <visual>
+                <origin rpy="0 0 0" xyz="0 0 0"/>
                 <geometry>
                     <mesh
@@ -125,4 +133,5 @@
         <link name="${prefix}robotiq_85_left_inner_knuckle_link">
             <visual>
+                <origin rpy="0 0 0" xyz="0 0 0"/>
                 <geometry>
                     <mesh
@@ -145,4 +154,5 @@
         <link name="${prefix}robotiq_85_right_inner_knuckle_link">
             <visual>
+                <origin rpy="0 0 0" xyz="0 0 0"/>
                 <geometry>
                     <mesh
@@ -165,4 +175,5 @@
         <link name="${prefix}robotiq_85_left_finger_tip_link">
             <visual>
+                <origin rpy="0 0 0" xyz="0 0 0"/>
                 <geometry>
                     <mesh
@@ -203,4 +214,5 @@
         <link name="${prefix}robotiq_85_right_finger_tip_link">
             <visual>
+                <origin rpy="0 0 0" xyz="0 0 0"/>
                 <geometry>
                     <mesh
