Commit message: Confirmed UR5e and Panda URDF files. Gotta change gazebo and robosuite ik for both if u wanna do something different

File: gazebo_env/description/urdf/hand_robosuite.xacro (robot description, xacro)
@@ -89,5 +89,5 @@
       <parent link="${ns}_hand"/>
       <child link="${ns}_ee"/>
-      <origin xyz="-0.004996500 -0.004996500 0.097724" rpy="0 0 0"/>
+      <origin xyz="-0.0000844170200 0.0000111528700 0.0964552948" rpy="0 0 0"/>
     </joint>
   </xacro:macro>

File: gazebo_env/description/urdf/panda_arm_hand_camera_scene_robosuite.urdf.xacro (robot description, xacro)
@@ -9,5 +9,6 @@
   <xacro:sensor_d435 parent="world">
     <!-- <origin xyz="1.613 0.032 1.441" rpy="0 0.2606116 3.14159" /> -->
-    <origin xyz="0.5 0 1.35" rpy="0 0.7840421 3.14159" />
+    <!-- for some reason we have to modify the xyz because it is a little shifted-->
+    <origin xyz="0.516 0.032 1.349" rpy="0 0.785398 3.14159" />
         <!-- <origin xyz="-1 0 0" rpy="0 3.1415927 1.5707963" /> -->
   </xacro:sensor_d435>

File: gazebo_env/description/urdf/ur5e_nvidia_with_gripper_camera_scene_robosuite.urdf.xacro (robot description, xacro)
@@ -7,5 +7,6 @@
   <xacro:include filename="$(find gazebo_env)/urdf/d435.urdf.xacro" />
   <xacro:sensor_d435 parent="world">
-    <origin xyz="1.488 1.534 1.496" rpy="0 0.6154831 -2.3561872" />
+    <origin xyz="0.516 0.032 1.349" rpy="0 0.785398 3.14159" />
+    <!-- <origin xyz="1.488 1.534 1.496" rpy="0 0.6154831 -2.3561872" /> -->
         <!-- <origin xyz="-1 0 0" rpy="0 3.1415927 1.5707963" /> -->
   </xacro:sensor_d435>

File: gazebo_env/description/urdf/ur5e_nvidia_with_gripper_robosuite.urdf.xacro (robot description, xacro)
@@ -502,5 +502,5 @@
     <link name="ur5e_ee_link" />
     <joint name="tool0_to_ur5e_ee_link_fixed_joint" type="fixed">
-      <origin rpy="0 0 0" xyz="0 0.001514 0.143" />
+      <origin rpy="0 0 0" xyz="0.000924756350 0.000929957310 0.142071136" />
       <parent link="tool0" />
       <child link="ur5e_ee_link" />
