Commit message: Switched to Trakikpy

File: gazebo_env/description/urdf/d435.urdf.xacro (robot description, xacro)
@@ -102,6 +102,6 @@
       <sensor name="camera" type="camera">
         <pose> 0 0 0 0 0 0 </pose>
-        <visualize>true</visualize>
-        <update_rate>10</update_rate>
+        <visualize>false</visualize>
+        <update_rate>30</update_rate>
         <camera>
             <horizontal_fov>1.089</horizontal_fov>

File: gazebo_env/description/urdf/ur5e_gazebo.urdf.xacro (robot description, xacro)
@@ -42,5 +42,5 @@
     <link name="world" />
     <xacro:sensor_d435 parent="world">
-        <origin xyz="1 1 0" rpy="0 0 -2.35619449" />
+        <origin xyz="1.5 1.5 1" rpy="0 0.5235987756 -2.35619449" />
     </xacro:sensor_d435>
     <joint name="base_joint" type="fixed">

Commit message: WE GOT EM

File: gazebo_env/description/urdf/d435.urdf.xacro (robot description, xacro)
@@ -105,9 +105,9 @@
         <update_rate>30</update_rate>
         <camera>
-            <horizontal_fov>1.089</horizontal_fov>
+            <horizontal_fov>0.7853981634</horizontal_fov>
             <image>
                 <format>R8G8B8</format>
-                <width>640</width>
-                <height>480</height>
+                <width>84</width>
+                <height>84</height>
             </image>
             <clip>

File: gazebo_env/description/urdf/panda_arm_hand_camera_scene_robosuite.urdf.xacro (robot description, xacro)
@@ -10,5 +10,5 @@
     <!-- <origin xyz="1.613 0.032 1.441" rpy="0 0.2606116 3.14159" /> -->
     <!-- for some reason we have to modify the xyz because it is a little shifted-->
-    <origin xyz="0.516 0.032 1.349" rpy="0 0.785398 3.14159" />
+    <origin xyz="0.516 0.018 1.349" rpy="0 0.7840421 3.1415927" />
         <!-- <origin xyz="-1 0 0" rpy="0 3.1415927 1.5707963" /> -->
   </xacro:sensor_d435>

Commit message: We got it better. Depth segmentation, no more pointclouds. We fast

File: gazebo_env/description/urdf/d435.urdf.xacro (robot description, xacro)
@@ -100,5 +100,5 @@
     <gazebo reference="camera_link">
       <material>Gazebo/TurquoiseGlowOutline </material>
-      <sensor name="camera" type="camera">
+      <sensor name="depth_camera" type="depth">
         <pose> 0 0 0 0 0 0 </pose>
         <visualize>false</visualize>

File: gazebo_env/description/urdf/panda_arm_hand_camera_scene_robosuite.urdf.xacro (robot description, xacro)
@@ -4,5 +4,5 @@
   <xacro:include filename="$(find gazebo_env)/urdf/hand_robosuite.xacro"/>
   <link name="world" />
-  <xacro:panda_arm connected_to="world" xyz="-0.56 0 0.912"/>
+  <xacro:panda_arm connected_to="world" xyz="-0.56 0 10.912"/>
   <xacro:hand ns="panda" rpy="0 0 ${-pi/4}" connected_to="panda_link8"/>
   <xacro:include filename="$(find gazebo_env)/urdf/d435.urdf.xacro" />
@@ -10,5 +10,5 @@
     <!-- <origin xyz="1.613 0.032 1.441" rpy="0 0.2606116 3.14159" /> -->
     <!-- for some reason we have to modify the xyz because it is a little shifted-->
-    <origin xyz="0.516 0.018 1.349" rpy="0 0.7840421 3.1415927" />
+    <origin xyz="0.516 0.018 11.349" rpy="0 0.7840421 3.1415927" />
         <!-- <origin xyz="-1 0 0" rpy="0 3.1415927 1.5707963" /> -->
   </xacro:sensor_d435>

Commit message: Lawrence has no warrants

File: gazebo_env/description/urdf/d435.urdf.xacro (robot description, xacro)
@@ -108,6 +108,8 @@
             <image>
                 <format>R8G8B8</format>
-                <width>84</width>
-                <height>84</height>
+                <width>256</width>
+                <height>256</height>
+                <!-- <width>256</width>
+                <height>256</height> -->
             </image>
             <clip>

File: gazebo_env/description/urdf/panda_arm_hand_camera_scene_robosuite.urdf.xacro (robot description, xacro)
@@ -4,12 +4,16 @@
   <xacro:include filename="$(find gazebo_env)/urdf/hand_robosuite.xacro"/>
   <link name="world" />
+  <!-- Lift task-->
   <xacro:panda_arm connected_to="world" xyz="-0.56 0 10.912"/>
+  <!-- Can task-->
+  <!-- <xacro:panda_arm connected_to="world" xyz="-0.56 -0.1 10.912"/>  -->
   <xacro:hand ns="panda" rpy="0 0 ${-pi/4}" connected_to="panda_link8"/>
   <xacro:include filename="$(find gazebo_env)/urdf/d435.urdf.xacro" />
   <xacro:sensor_d435 parent="world">
-    <!-- <origin xyz="1.613 0.032 1.441" rpy="0 0.2606116 3.14159" /> -->
     <!-- for some reason we have to modify the xyz because it is a little shifted-->
+    <!-- Lift task-->
     <origin xyz="0.516 0.018 11.349" rpy="0 0.7840421 3.1415927" />
-        <!-- <origin xyz="-1 0 0" rpy="0 3.1415927 1.5707963" /> -->
+    <!-- Can task-->
+    <!-- <origin xyz="1.016 0.018 11.749" rpy="0 0.7840421 3.1415927" />  -->
   </xacro:sensor_d435>
   <gazebo>
