Commit message: Think Panda works

File: gazebo_env/description/urdf/panda_ik_robosuite.urdf (robot description, URDF)
Before this commit: robot panda, 14 links, 13 joints
Links:
- link panda_hand: geometry 
- link panda_leftfinger: geometry 
- link panda_link0: geometry 
- link panda_link1: geometry 
- link panda_link2: geometry 
- link panda_link3: geometry 
- link panda_link4: geometry 
- link panda_link5: geometry 
- link panda_link6: geometry 
- link panda_link7: geometry 
- link panda_rightfinger: geometry 

File: gazebo_env/description/urdf/ur5e_ik_robosuite.urdf (robot description, URDF)
Before this commit: robot ur5e_scene, 20 links, 19 joints
Links:
- link base_link: geometry 
- link forearm_link: geometry 
- link robotiq_85_base_link: geometry 
- link robotiq_85_left_finger_link: geometry 
- link robotiq_85_left_finger_tip_link: geometry 
- link robotiq_85_left_inner_knuckle_link: geometry 
- link robotiq_85_left_knuckle_link: geometry 
- link robotiq_85_right_finger_link: geometry 
- link robotiq_85_right_finger_tip_link: geometry 
- link robotiq_85_right_inner_knuckle_link: geometry 
- link robotiq_85_right_knuckle_link: geometry 
- link shoulder_link: geometry 
- link upper_arm_link: geometry 
- link wrist_1_link: geometry 
- link wrist_2_link: geometry 
- link wrist_3_link: geometry 
