Commit message: Added UR5 robot in Gazebo

File: gazebo_env/description/urdf/panda_arm_hand_camera_scene_real.urdf.xacro (robot description, xacro)
@@ -9,9 +9,8 @@
   <!-- <xacro:panda_arm connected_to="world" xyz="-0.56 -0.1 10.912"/>  -->
   <xacro:hand ns="panda" rpy="0 0 ${-pi/4}" connected_to="panda_link8"/>
-  <xacro:include filename="$(find gazebo_env)/urdf/d435.urdf.xacro" />
   <!-- Can task-->
   <!-- <xacro:panda_arm connected_to="world" xyz="-0.56 -0.1 10.912"/>  -->
   <!-- <xacro:hand ns="panda" rpy="0 0 ${-pi/4}" connected_to="panda_link8"/> -->
-  <xacro:include filename="$(find gazebo_env)/urdf/real_cam.urdf.xacro" />
+  <xacro:include filename="$(find gazebo_env)/urdf/real_panda_cam.urdf.xacro" />
   <xacro:sensor_d435 parent="world">
     <!-- for some reason we have to modify the xyz because it is a little shifted-->

File: gazebo_env/description/urdf/panda_arm_hand_ur5e_gripper_camera_scene_real.urdf.xacro (robot description, xacro)
@@ -8,11 +8,10 @@
   <!-- <xacro:panda_arm connected_to="world" xyz="-0.56 -0.1 10.912"/>  -->
   <!-- <xacro:hand ns="panda" rpy="0 0 ${-pi/4}" connected_to="panda_link8"/> -->
-  <xacro:include filename="$(find gazebo_env)/urdf/real_cam.urdf.xacro" />
+  <xacro:include filename="$(find gazebo_env)/urdf/real_panda_cam.urdf.xacro" />
+  <!-- <xacro:sensor_d435 parent="world">
+    <origin xyz="0.84531124 0.0494013 10.61637858" rpy="0.0381616 0.6288943 -3.0232923" />
+  </xacro:sensor_d435> -->
   <xacro:sensor_d435 parent="world">
-    <!-- for some reason we have to modify the xyz because it is a little shifted-->
-    <!-- Lift task-->
-    <origin xyz="0.84531124 0.0494013 10.61637858" rpy="0.0381616 0.6288943 -3.0232923" />
-    <!-- Can task-->
-    <!-- <origin xyz="1.016 0.018 11.749" rpy="0 0.7840421 3.1415927" />  -->
+    <origin xyz="0.90641516 -0.08090482 10.6424972" rpy="0.0588804 0.6888795 3.1219407" />
   </xacro:sensor_d435>
   <gazebo>
