Commit message: First crack at real online setup

File: gazebo_env/description/urdf/panda_arm_hand_ur5e_gripper_camera_scene_real.urdf.xacro (robot description, xacro)
@@ -2,20 +2,28 @@
 <robot xmlns:xacro="http://www.ros.org/wiki/xacro" name="panda">
   <xacro:include filename="$(find gazebo_env)/urdf/panda_arm_ur5e_gripper.xacro"/>
+  <xacro:include filename="$(find gazebo_env)/urdf/ur5_with_gripper.urdf.xacro" />
   <link name="world" />
   <!-- Lift task-->
-  <xacro:panda_arm connected_to="world" xyz="0 0 10"/>
+  <!-- <xacro:panda_arm connected_to="world" xyz="0 0 10"/>  -->
   <!-- Can task-->
   <!-- <xacro:panda_arm connected_to="world" xyz="-0.56 -0.1 10.912"/>  -->
   <!-- <xacro:hand ns="panda" rpy="0 0 ${-pi/4}" connected_to="panda_link8"/> -->
-  <xacro:include filename="$(find gazebo_env)/urdf/real_panda_cam.urdf.xacro" />
-  <!-- <xacro:sensor_d435 parent="world">
+  <!-- <xacro:include filename="$(find gazebo_env)/urdf/real_panda_cam.urdf.xacro" /> -->
+  <!-- <xacro:sensor_d435_panda parent="world">
     <origin xyz="0.84531124 0.0494013 10.61637858" rpy="0.0381616 0.6288943 -3.0232923" />
-  </xacro:sensor_d435> -->
-  <xacro:sensor_d435 parent="world">
-    <origin xyz="0.90641516 -0.08090482 10.6424972" rpy="0.0588804 0.6888795 3.1219407" />
-  </xacro:sensor_d435>
-  <gazebo>
+  </xacro:sensor_d435_panda> -->
+  <!-- <xacro:sensor_d435_panda parent="world"> -->
+    <!-- <origin xyz="0.90641516 -0.08090482 10.6424972" rpy="0.0588804 0.6888795 3.1219407" /> -->
+  <!-- </xacro:sensor_d435_panda> -->
+  <xacro:ur5e_gripper parent="world">
+      <origin xyz="10 0 10" rpy="0 0 0" />
+  </xacro:ur5e_gripper>
+  <xacro:include filename="$(find gazebo_env)/urdf/real_ur5_cam.urdf.xacro" />
+  <xacro:sensor_d435_ur5 parent="world">
+    <origin xyz="10.90641516 -0.08090482 10.6424972" rpy="0.0588804 0.6888795 3.1219407" />
+  </xacro:sensor_d435_ur5>
+  <!-- <gazebo>
     <plugin name="no_physics" filename="libno_physics_plugin.so" />
-  </gazebo>
+  </gazebo> -->
   <gazebo>
     <plugin name="panda_control_real" filename="libpanda_control_ur5e_gripper_real_plugin.so" />

File: gazebo_env/description/urdf/real_panda_cam.urdf.xacro (robot description, xacro)
@@ -5,24 +5,24 @@
 <!-- =================================================================================== -->
 <robot name="realsense2_camera" xmlns:xacro="http://ros.org/wiki/xacro">
-  <xacro:macro name="sensor_d435"
+  <xacro:macro name="sensor_d435_panda"
     params="parent *origin name:=camera use_nominal_extrinsics:=false add_plug:=false use_mesh:=true">
-    <material name="aluminum">
+    <material name="panda_aluminum">
       <color rgba="0.5 0.5 0.5 1" />
     </material>
-    <material name="plastic">
+    <material name="panda_plastic">
       <color rgba="0.1 0.1 0.1 1" />
     </material>
-    <joint name="camera_joint" type="fixed">
+    <joint name="panda_camera_joint" type="fixed">
       <xacro:insert_block name="origin" />
       <parent link="${parent}" />
-      <child link="camera_bottom_screw_frame" />
+      <child link="panda_camera_bottom_screw_frame" />
     </joint>
-    <link name="camera_bottom_screw_frame" />
-    <joint name="camera_link_joint" type="fixed">
+    <link name="panda_camera_bottom_screw_frame" />
+    <joint name="panda_camera_link_joint" type="fixed">
       <origin rpy="0 0 0" xyz="0.010600000000000002 0.0175 0.0125" />
-      <parent link="camera_bottom_screw_frame" />
-      <child link="camera_link" />
+      <parent link="panda_camera_bottom_screw_frame" />
+      <child link="panda_camera_link" />
     </joint>
-    <link name="camera_link">
+    <link name="panda_camera_link">
       <visual>
         <!-- the mesh origin is at front plate in between the two infrared camera axes -->
@@ -47,58 +47,58 @@
     </link>
     <!-- camera depth joints and links -->
-    <joint name="camera_depth_joint" type="fixed">
+    <joint name="panda_camera_depth_joint" type="fixed">
       <origin rpy="0 0 0" xyz="0 0 0" />
-      <parent link="camera_link" />
-      <child link="camera_depth_frame" />
+      <parent link="panda_camera_link" />
+      <child link="panda_camera_depth_frame" />
     </joint>
-    <link name="camera_depth_frame" />
-    <joint name="camera_depth_optical_joint" type="fixed">
+    <link name="panda_camera_depth_frame" />
+    <joint name="panda_camera_depth_optical_joint" type="fixed">
       <origin rpy="-1.5707963267948966 0 -1.5707963267948966" xyz="0 0 0" />
-      <parent link="camera_depth_frame" />
-      <child link="camera_depth_optical_frame" />
+      <parent link="panda_camera_depth_frame" />
+      <child link="panda_camera_depth_optical_frame" />
     </joint>
-    <link name="camera_depth_optical_frame" />
+    <link name="panda_camera_depth_optical_frame" />
     <!-- camera left IR joints and links -->
-    <joint name="camera_infra1_joint" type="fixed">
+    <joint name="panda_camera_infra1_joint" type="fixed">
       <origin rpy="0 0 0" xyz="0 0.0 0" />
-      <parent link="camera_link" />
-      <child link="camera_infra1_frame" />
+      <parent link="panda_camera_link" />
+      <child link="panda_camera_infra1_frame" />
     </joint>
-    <link name="camera_infra1_frame" />
-    <joint name="camera_infra1_optical_joint" type="fixed">
+    <link name="panda_camera_infra1_frame" />
+    <joint name="panda_camera_infra1_optical_joint" type="fixed">
       <origin rpy="-1.5707963267948966 0 -1.5707963267948966" xyz="0 0 0" />
-      <parent link="camera_infra1_frame" />
-      <child link="camera_infra1_optical_frame" />
+      <parent link="panda_camera_infra1_frame" />
+      <child link="panda_camera_infra1_optical_frame" />
     </joint>
-    <link name="camera_infra1_optical_frame" />
+    <link name="panda_camera_infra1_optical_frame" />
     <!-- camera right IR joints and links -->
-    <joint name="camera_infra2_joint" type="fixed">
+    <joint name="panda_camera_infra2_joint" type="fixed">
       <origin rpy="0 0 0" xyz="0 -0.05 0" />
-      <parent link="camera_link" />
-      <child link="camera_infra2_frame" />
+      <parent link="panda_camera_link" />
+      <child link="panda_camera_infra2_frame" />
     </joint>
-    <link name="camera_infra2_frame" />
-    <joint name="camera_infra2_optical_joint" type="fixed">
+    <link name="panda_camera_infra2_frame" />
+    <joint name="panda_camera_infra2_optical_joint" type="fixed">
       <origin rpy="-1.5707963267948966 0 -1.5707963267948966" xyz="0 0 0" />
-      <parent link="camera_infra2_frame" />
-      <child link="camera_infra2_optical_frame" />
+      <parent link="panda_camera_infra2_frame" />
+      <child link="panda_camera_infra2_optical_frame" />
     </joint>
-    <link name="camera_infra2_optical_frame" />
+    <link name="panda_camera_infra2_optical_frame" />
     <!-- camera color joints and links -->
-    <joint name="camera_color_joint" type="fixed">
+    <joint name="panda_camera_color_joint" type="fixed">
       <origin rpy="0 0 0" xyz="0 0.015 0" />
-      <parent link="camera_link" />
-      <child link="camera_color_frame" />
+      <parent link="panda_camera_link" />
+      <child link="panda_camera_color_frame" />
     </joint>
-    <link name="camera_color_frame" />
-    <joint name="camera_color_optical_joint" type="fixed">
+    <link name="panda_camera_color_frame" />
+    <joint name="panda_camera_color_optical_joint" type="fixed">
       <origin rpy="-1.5707963267948966 0 -1.5707963267948966" xyz="0 0 0" />
-      <parent link="camera_color_frame" />
-      <child link="camera_color_optical_frame" />
+      <parent link="panda_camera_color_frame" />
+      <child link="panda_camera_color_optical_frame" />
     </joint>
-    <link name="camera_color_optical_frame" />
-    <gazebo reference="camera_link">
+    <link name="panda_camera_color_optical_frame" />
+    <gazebo reference="panda_camera_link">
       <material>Gazebo/TurquoiseGlowOutline </material>
-      <sensor name="depth_camera" type="depth">
+      <sensor name="panda_camera" type="depth">
         <pose> 0 0 0 0 0 0 </pose>
         <visualize>false</visualize>
@@ -119,6 +119,6 @@
             </clip>
         </camera>
-        <plugin name="camera_controller" filename="libgazebo_ros_camera.so">
-            <frame_name>camera_color_optical_frame</frame_name>
+        <plugin name="panda_camera_controller" filename="libgazebo_ros_camera.so">
+            <frame_name>panda_camera_color_optical_frame</frame_name>
             <!-- <cx>647.53735352</cx> -->
             <!-- <cy>367.65203857</cy> -->

File: gazebo_env/description/urdf/real_ur5_cam.urdf.xacro (robot description, xacro)
@@ -5,24 +5,24 @@
 <!-- =================================================================================== -->
 <robot name="realsense2_camera" xmlns:xacro="http://ros.org/wiki/xacro">
-  <xacro:macro name="sensor_d435"
+  <xacro:macro name="sensor_d435_ur5"
     params="parent *origin name:=camera use_nominal_extrinsics:=false add_plug:=false use_mesh:=true">
-    <material name="aluminum">
+    <material name="ur5_aluminum">
       <color rgba="0.5 0.5 0.5 1" />
     </material>
-    <material name="plastic">
+    <material name="ur5_plastic">
       <color rgba="0.1 0.1 0.1 1" />
     </material>
-    <joint name="camera_joint" type="fixed">
+    <joint name="ur5_camera_joint" type="fixed">
       <xacro:insert_block name="origin" />
       <parent link="${parent}" />
-      <child link="camera_bottom_screw_frame" />
+      <child link="ur5_camera_bottom_screw_frame" />
     </joint>
-    <link name="camera_bottom_screw_frame" />
-    <joint name="camera_link_joint" type="fixed">
+    <link name="ur5_camera_bottom_screw_frame" />
+    <joint name="ur5_camera_link_joint" type="fixed">
       <origin rpy="0 0 0" xyz="0.010600000000000002 0.0175 0.0125" />
-      <parent link="camera_bottom_screw_frame" />
-      <child link="camera_link" />
+      <parent link="ur5_camera_bottom_screw_frame" />
+      <child link="ur5_camera_link" />
     </joint>
-    <link name="camera_link">
+    <link name="ur5_camera_link">
       <visual>
         <!-- the mesh origin is at front plate in between the two infrared camera axes -->
@@ -47,58 +47,58 @@
     </link>
     <!-- camera depth joints and links -->
-    <joint name="camera_depth_joint" type="fixed">
+    <joint name="ur5_camera_depth_joint" type="fixed">
       <origin rpy="0 0 0" xyz="0 0 0" />
-      <parent link="camera_link" />
-      <child link="camera_depth_frame" />
+      <parent link="ur5_camera_link" />
+      <child link="ur5_camera_depth_frame" />
     </joint>
-    <link name="camera_depth_frame" />
-    <joint name="camera_depth_optical_joint" type="fixed">
+    <link name="ur5_camera_depth_frame" />
+    <joint name="ur5_camera_depth_optical_joint" type="fixed">
       <origin rpy="-1.5707963267948966 0 -1.5707963267948966" xyz="0 0 0" />
-      <parent link="camera_depth_frame" />
-      <child link="camera_depth_optical_frame" />
+      <parent link="ur5_camera_depth_frame" />
+      <child link="ur5_camera_depth_optical_frame" />
     </joint>
-    <link name="camera_depth_optical_frame" />
+    <link name="ur5_camera_depth_optical_frame" />
     <!-- camera left IR joints and links -->
-    <joint name="camera_infra1_joint" type="fixed">
+    <joint name="ur5_camera_infra1_joint" type="fixed">
       <origin rpy="0 0 0" xyz="0 0.0 0" />
-      <parent link="camera_link" />
-      <child link="camera_infra1_frame" />
+      <parent link="ur5_camera_link" />
+      <child link="ur5_camera_infra1_frame" />
     </joint>
-    <link name="camera_infra1_frame" />
-    <joint name="camera_infra1_optical_joint" type="fixed">
+    <link name="ur5_camera_infra1_frame" />
+    <joint name="ur5_camera_infra1_optical_joint" type="fixed">
       <origin rpy="-1.5707963267948966 0 -1.5707963267948966" xyz="0 0 0" />
-      <parent link="camera_infra1_frame" />
-      <child link="camera_infra1_optical_frame" />
+      <parent link="ur5_camera_infra1_frame" />
+      <child link="ur5_camera_infra1_optical_frame" />
     </joint>
-    <link name="camera_infra1_optical_frame" />
+    <link name="ur5_camera_infra1_optical_frame" />
     <!-- camera right IR joints and links -->
-    <joint name="camera_infra2_joint" type="fixed">
+    <joint name="ur5_camera_infra2_joint" type="fixed">
       <origin rpy="0 0 0" xyz="0 -0.05 0" />
-      <parent link="camera_link" />
-      <child link="camera_infra2_frame" />
+      <parent link="ur5_camera_link" />
+      <child link="ur5_camera_infra2_frame" />
     </joint>
-    <link name="camera_infra2_frame" />
-    <joint name="camera_infra2_optical_joint" type="fixed">
+    <link name="ur5_camera_infra2_frame" />
+    <joint name="ur5_camera_infra2_optical_joint" type="fixed">
       <origin rpy="-1.5707963267948966 0 -1.5707963267948966" xyz="0 0 0" />
-      <parent link="camera_infra2_frame" />
-      <child link="camera_infra2_optical_frame" />
+      <parent link="ur5_camera_infra2_frame" />
+      <child link="ur5_camera_infra2_optical_frame" />
     </joint>
-    <link name="camera_infra2_optical_frame" />
+    <link name="ur5_camera_infra2_optical_frame" />
     <!-- camera color joints and links -->
-    <joint name="camera_color_joint" type="fixed">
+    <joint name="ur5_camera_color_joint" type="fixed">
       <origin rpy="0 0 0" xyz="0 0.015 0" />
-      <parent link="camera_link" />
-      <child link="camera_color_frame" />
+      <parent link="ur5_camera_link" />
+      <child link="ur5_camera_color_frame" />
     </joint>
-    <link name="camera_color_frame" />
-    <joint name="camera_color_optical_joint" type="fixed">
+    <link name="ur5_camera_color_frame" />
+    <joint name="ur5_camera_color_optical_joint" type="fixed">
       <origin rpy="-1.5707963267948966 0 -1.5707963267948966" xyz="0 0 0" />
-      <parent link="camera_color_frame" />
-      <child link="camera_color_optical_frame" />
+      <parent link="ur5_camera_color_frame" />
+      <child link="ur5_camera_color_optical_frame" />
     </joint>
-    <link name="camera_color_optical_frame" />
-    <gazebo reference="camera_link">
+    <link name="ur5_camera_color_optical_frame" />
+    <gazebo reference="ur5_camera_link">
       <material>Gazebo/TurquoiseGlowOutline </material>
-      <sensor name="depth_camera" type="depth">
+      <sensor name="ur5_camera" type="depth">
         <pose> 0 0 0 0 0 0 </pose>
         <visualize>false</visualize>
@@ -119,6 +119,6 @@
             </clip>
         </camera>
-        <plugin name="camera_controller" filename="libgazebo_ros_camera.so">
-            <frame_name>camera_color_optical_frame</frame_name>
+        <plugin name="ur5_camera_controller" filename="libgazebo_ros_camera.so">
+            <frame_name>ur5_camera_color_optical_frame</frame_name>
             <!-- <cx>647.53735352</cx> -->
             <!-- <cy>367.65203857</cy> -->

File: gazebo_env/description/urdf/ur5_with_gripper_and_panda_camera_scene_real.urdf.xacro (robot description, xacro)
@@ -1,27 +1,28 @@
-<?xml version="1.0" encoding="utf-8"?>
-<robot xmlns:xacro="http://www.ros.org/wiki/xacro" name="panda">
+<robot name="ur5e_scene" xmlns:xacro="http://ros.org/wiki/xacro">
+  <xacro:include filename="$(find gazebo_env)/urdf/ur5_with_gripper.urdf.xacro" />
   <xacro:include filename="$(find gazebo_env)/urdf/panda_arm.xacro"/>
   <xacro:include filename="$(find gazebo_env)/urdf/hand_robosuite.xacro"/>
   <link name="world" />
+  <xacro:ur5e_gripper parent="world">
+      <origin xyz="0 0 10" rpy="0 0 0" />
+  </xacro:ur5e_gripper>
+  <xacro:include filename="$(find gazebo_env)/urdf/real_ur5_cam.urdf.xacro" />
+  <xacro:sensor_d435_ur5 parent="world">
+    <origin xyz="0.90641516 -0.08090482 10.6424972" rpy="0.0588804 0.6888795 3.1219407" />
+  </xacro:sensor_d435_ur5>
   <!-- Lift task-->
-  <xacro:panda_arm connected_to="world" xyz="0 0 10"/>
+  <xacro:panda_arm connected_to="world" xyz="10 0 10"/>
   <!-- Can task-->
   <!-- <xacro:panda_arm connected_to="world" xyz="-0.56 -0.1 10.912"/>  -->
   <xacro:hand ns="panda" rpy="0 0 ${-pi/4}" connected_to="panda_link8"/>
-  <!-- Can task-->
-  <!-- <xacro:panda_arm connected_to="world" xyz="-0.56 -0.1 10.912"/>  -->
-  <!-- <xacro:hand ns="panda" rpy="0 0 ${-pi/4}" connected_to="panda_link8"/> -->
   <xacro:include filename="$(find gazebo_env)/urdf/real_panda_cam.urdf.xacro" />
   <xacro:sensor_d435_panda parent="world">
     <!-- for some reason we have to modify the xyz because it is a little shifted-->
     <!-- Lift task-->
-    <origin xyz="0.84531124 0.0494013 10.61637858" rpy="0.0381616 0.6288943 -3.0232923" />
+    <origin xyz="10.84531124 0.0494013 10.61637858" rpy="0.0381616 0.6288943 -3.0232923" />
     <!-- Can task-->
     <!-- <origin xyz="1.016 0.018 11.749" rpy="0 0.7840421 3.1415927" />  -->
   </xacro:sensor_d435_panda>
   <gazebo>
-    <plugin name="no_physics" filename="libno_physics_plugin.so" />
-  </gazebo>
-  <gazebo>
     <plugin name="panda_control" filename="libpanda_control_plugin.so" />
   </gazebo>

File: gazebo_env/description/urdf/ur5_with_gripper_camera_scene_real.urdf.xacro (robot description, xacro)
@@ -5,7 +5,7 @@
       <origin xyz="0 0 10" rpy="0 0 0" />
   </xacro:ur5e_gripper>
-  <xacro:include filename="$(find gazebo_env)/urdf/real_ur5e_cam.urdf.xacro" />
-  <xacro:sensor_d435 parent="world">
+  <xacro:include filename="$(find gazebo_env)/urdf/real_ur5_cam.urdf.xacro" />
+  <xacro:sensor_d435_ur5 parent="world">
     <origin xyz="0.90641516 -0.08090482 10.6424972" rpy="0.0588804 0.6888795 3.1219407" />
-  </xacro:sensor_d435>
+  </xacro:sensor_d435_ur5>
 </robot>
