Commit message: Setup real experiments, and sim experiments. Along with camera deprojection and reprojection

File: gazebo_env/description/urdf/ur5_and_panda_gripper_camera_scene_real.urdf.xacro (robot description, xacro)
@@ -1,9 +1,10 @@
 <robot name="ur5e_scene" xmlns:xacro="http://ros.org/wiki/xacro">
-  <xacro:include filename="$(find gazebo_env)/urdf/ur5.urdf.xacro" />
+  <xacro:include filename="$(find gazebo_env)/urdf/ur5_with_gripper.urdf.xacro" />
   <xacro:include filename="$(find gazebo_env)/urdf/panda_arm.xacro"/>
+  <xacro:include filename="$(find gazebo_env)/urdf/hand.xacro"/>
   <link name="world" />
-  <xacro:ur5 parent="world">
+  <xacro:ur5_gripper parent="world">
       <origin xyz="0 0 10" rpy="0 0 0" />
-  </xacro:ur5>
+  </xacro:ur5_gripper>
   <xacro:include filename="$(find gazebo_env)/urdf/real_ur5_cam.urdf.xacro" />
   <xacro:sensor_d435_ur5 parent="world">
@@ -12,4 +13,5 @@
   <!-- Lift task-->
   <xacro:panda_arm connected_to="world" xyz="10 0 10"/>
+  <xacro:hand ns="panda" rpy="0 0 0" connected_to="panda_link8"/>
   <!-- Can task-->
   <!-- <xacro:panda_arm connected_to="world" xyz="-0.56 -0.1 10.912"/>  -->
@@ -23,5 +25,5 @@
   </xacro:sensor_d435_panda>
   <gazebo>
-    <plugin name="ur5_and_panda_no_gripper_control" filename="libur5_and_panda_no_gripper_control_plugin.so" />
+    <plugin name="ur5_and_panda_gripper_control" filename="libur5_and_panda_gripper_control_plugin.so" />
   </gazebo>
   <gazebo>

File: gazebo_env/description/urdf/ur5_with_gripper.urdf.xacro (robot description, xacro)
@@ -4,7 +4,7 @@
 <!-- |    EDITING THIS FILE BY HAND IS NOT RECOMMENDED                                 | -->
 <!-- =================================================================================== -->
-<robot name="ur5e_gripper" xmlns:xacro="http://ros.org/wiki/xacro">
-  <xacro:macro name="ur5e_gripper"
-    params="parent:=world *origin name:=ur5e_gripper">
+<robot name="ur5_gripper" xmlns:xacro="http://ros.org/wiki/xacro">
+  <xacro:macro name="ur5_gripper"
+    params="parent:=world *origin name:=ur5_gripper">
     <joint name="base_joint" type="fixed">
       <xacro:insert_block name="origin" />
@@ -1084,10 +1084,10 @@
       <plugin name="ur5e_control" filename="libur5e_control_plugin.so" />
     </gazebo> -->
-    <gazebo>
+    <!-- <gazebo>
       <plugin name="no_physics" filename="libno_physics_plugin.so" />
     </gazebo>
     <gazebo>
       <plugin name="ur5e_control" filename="libur5e_control_plugin.so" />
-    </gazebo>
+    </gazebo> -->
   </xacro:macro>
 </robot>
